Commit message: Correct stereo camera orientation and placement.

File: hector_quadrotor_description/urdf/quadrotor_downward_cam.urdf.xacro (robot description, xacro)
@@ -19,4 +19,4 @@
                        noise_stddev="0.015"
                        update_rate="1"
-                       off_x="0.5" off_y="-0.15" off_z="0.0" />
+                       off_x="0.15" off_y="0.0" off_z="-0.10" />
 </robot>

File: hector_quadrotor_description/urdf/stereo_mast-triggered.xacro (robot description, xacro)
@@ -36,5 +36,5 @@
     <parent link="${stereo_mast_parent_link}"/>
     <child link="${Camera01Name}_mast_link"/>
-    <origin xyz="${off_x} ${off_y} ${off_z}" rpy="${pi} 0 0" />
+    <origin xyz="${off_x} ${off_y} ${off_z}" rpy="${pi} ${pi/2} 0" />
   </joint>
   <link name="${Camera01Name}_head_link">
