Commit message: disabling quad in urdf instead of sdf.. this is more general...

File: hector_quadrotor_description/urdf/quadrotor_base_slave.urdf.xacro (robot description, xacro)
@@ -1,5 +1,4 @@
 <?xml version="1.0"?>
 <robot xmlns:xacro="http://www.ros.org/wiki/xacro">
-  <xacro:include filename="$(find hector_sensors_description)/urdf/sonar_sensor.urdf.xacro" />
   <xacro:property name="pi" value="3.1415926535897931" />
   <!-- Main quadrotor link -->
@@ -24,8 +23,4 @@
       </collision>
     </link>
-    <!-- Sonar height sensor -->
-    <xacro:sonar_sensor name="sonar" parent="base_link" ros_topic="sonar_height" update_rate="10" min_range="0.03" max_range="3.0" field_of_view="${40*pi/180}" ray_count="3">
-      <origin xyz="-0.16 0.0 -0.012" rpy="0 ${90*pi/180} 0"/>
-    </xacro:sonar_sensor>
   </xacro:macro>
 </robot>

File: hector_quadrotor_description/urdf/quadrotor_downward_cam_slave.urdf.xacro (robot description, xacro)
@@ -4,9 +4,11 @@
     <!-- Included URDF Files -->
     <xacro:include filename="$(find hector_quadrotor_description)/urdf/quadrotor_base_slave.urdf.xacro" />
+    <xacro:include filename="$(find hector_quadrotor_description)/urdf/disable_quad_slave.urdf.xacro" />
     <!-- Instantiate quadrotor_base_slave_macro once (has no parameters atm) -->
     <xacro:quadrotor_base_slave_macro />
+    <xacro:disable_quad_slave_macro />
     <!-- Downward facing camera -->
     <xacro:include filename="$(find hector_sensors_description)/urdf/generic_camera.urdf.xacro" />
-    <xacro:generic_camera name="downward_cam" parent="base_link" ros_topic="camera/image" cam_info_topic="camera/camera_info" update_rate="20" res_x="640" res_y="480" image_format="R8G8B8" hfov="100">
+    <xacro:generic_camera name="downward_cam_slave_01" parent="base_link" ros_topic="camera/image_slave_01" cam_info_topic="camera/camera_info_slave_01" update_rate="20" res_x="640" res_y="480" image_format="R8G8B8" hfov="100">
       <origin xyz="0.4 0.0 -0.0" rpy="0 ${M_PI/2} 0"/>
     </xacro:generic_camera>
