Commit message: Edited downward camera frame rate

File: hector_quadrotor_description/urdf/quadrotor_downward_cam.gazebo.xacro (robot description, xacro)
@@ -3,4 +3,4 @@
     <xacro:include filename="$(find hector_quadrotor_description)/urdf/quadrotor_downward_cam.urdf.xacro" />
     <xacro:include filename="$(find hector_quadrotor_gazebo)/urdf/quadrotor_plugins.gazebo.xacro" />
-    <xacro:quadrotor_plugins />
+	<xacro:macro name="quadrotor_plugins"></xacro:macro>
 </robot>

File: hector_quadrotor_description/urdf/quadrotor_downward_cam.urdf.xacro (robot description, xacro)
@@ -6,8 +6,13 @@
     <!-- Instantiate quadrotor_base_macro once (has no parameters atm) -->
     <xacro:quadrotor_base_macro />
-    <!-- Downward facing camera -->
-    <xacro:include filename="$(find hector_sensors_description)/urdf/generic_camera.urdf.xacro" />
+    <!-- Downward facing camera: Original configuration -->
+    <!--xacro:include filename="$(find hector_sensors_description)/urdf/generic_camera.urdf.xacro" />
     <xacro:generic_camera name="downward_cam" parent="base_link" ros_topic="camera/image" cam_info_topic="camera/camera_info" update_rate="20" res_x="640" res_y="480" image_format="R8G8B8" hfov="100">
       <origin xyz="0.4 0.0 -0.0" rpy="0 ${M_PI/2} 0"/>
+    </xacro:generic_camera -->
+        <!-- Downward facing camera -->
+    <xacro:include filename="$(find hector_sensors_description)/urdf/generic_camera.urdf.xacro" />
+    <xacro:generic_camera name="downward_cam" parent="base_link" ros_topic="camera/image" cam_info_topic="camera/camera_info" update_rate="1" res_x="640" res_y="480" image_format="R8G8B8" hfov="100">
+      <origin xyz="0.4 0.0 0.0" rpy="0 ${M_PI/2} 0"/>
     </xacro:generic_camera>
 </robot>
