Commit message: Committing before a merge

File: hector_quadrotor_gazebo/urdf/quadrotor_plugins.gazebo.xacro (robot description, xacro)
@@ -7,10 +7,8 @@
   <xacro:include filename="$(find hector_quadrotor_gazebo)/urdf/quadrotor_propulsion.gazebo.xacro" />
   <xacro:include filename="$(find hector_quadrotor_gazebo)/urdf/quadrotor_aerodynamics.gazebo.xacro" />
-	<!-- Quadrotor Gazebo Plugins -->
-	<xacro:macro name="quadrotor_plugins">
+  <!-- Quadrotor Gazebo Plugins -->
   <xacro:quadrotor_sensors />
   <xacro:quadrotor_controller />
   <xacro:quadrotor_propulsion />
-	<xacro:quadrotor_aerodynamics />
-</xacro:macro>
+  <xacro:quadrotor_aerodynamics />
 </robot>

Commit message: Update controller parameters to fly smoothlier

File: hector_quadrotor_gazebo/urdf/quadrotor_plugins.gazebo.xacro (robot description, xacro)
@@ -7,10 +7,9 @@
   <xacro:include filename="$(find hector_quadrotor_gazebo)/urdf/quadrotor_propulsion.gazebo.xacro" />
   <xacro:include filename="$(find hector_quadrotor_gazebo)/urdf/quadrotor_aerodynamics.gazebo.xacro" />
-	<!-- Quadrotor Gazebo Plugins -->
-	<xacro:macro name="quadrotor_plugins">
+  <!-- Quadrotor Gazebo Plugins -->
   <xacro:quadrotor_sensors />
   <xacro:quadrotor_controller />
   <xacro:quadrotor_propulsion />
-	<xacro:quadrotor_aerodynamics />
-</xacro:macro>
+  <xacro:quadrotor_aerodynamics />
+  <xacro:macro name="quadrotor_plugins"></xacro:macro>
 </robot>
